File: KiCad Files/custom_keyboard.sch (KiCad schematic (older format))
At the start: 28 parts

Commit message: keys in schematic
Parts:
- removed C?: 1u, symbol Device:C
- removed C? (x3): 0.1u, symbol Device:C
- removed C?: 10u, symbol Device:C
- removed R? (x2): 10k, symbol Device:R
- removed SW?: SW_Push, symbol Switch:SW_Push
- removed U?: ATmega32U4-AU, Package_QFP:TQFP-44_10x10mm_P0.8mm, symbol MCU_Microchip_ATmega:ATmega32U4-AU
- added C1, C2: 10u, Capacitor_SMD:C_0805_2012Metric, symbol Device:CP
- added C10, C11, C12, C13, C7, C9: 100n, Capacitor_SMD:C_0805_2012Metric, symbol Device:C
- added C3: 0.1u, Capacitor_SMD:C_0805_2012Metric, symbol Device:C
- added C6, C8: 4.7u, Capacitor_SMD:C_0805_2012Metric, symbol Device:C
- added D1, D101, D102, D103, D105, D107, D108, D110, D111, D113, D115, D116, D117, D119, D12, D120, D121, D123, D125, D126, D127, D129, D130, D131, D14, D17, D19, D20, D22, D24, D25, D27, D28, D3, D30, D32, D33, D35, D36, D38, D4, D40, D41, D43, D44, D46, D48, D5, D50, D51, D52, D54, D56, D58, D60, D61, D62, D64, D66, D68, D69, D70, D72, D73, D76, D77, D78, D80, D82, D84, D85, D87, D89, D9, D91, D92, D94, D95, D97, D99: D_Small, Diode_SMD:D_SOD-123, symbol Device:D_Small
- added J1: Conn_01x05_Male, Connector_PinHeader_2.54mm:PinHeader_1x05_P2.54mm_Vertical, symbol Connector:Conn_01x05_Male
- added MX1: MX-NoLED L SHIFT, Button_Switch_Keyboard:SW_Cherry_MX_2.25u_PCB, symbol MX_Alps_Hybrid:MX-NoLED
- added MX10: MX-NoLED A, Button_Switch_Keyboard:SW_Cherry_MX_1.00u_PCB, symbol MX_Alps_Hybrid:MX-NoLED
- added MX12, MX57: MX-NoLED ALT, Button_Switch_Keyboard:SW_Cherry_MX_1.25u_PCB, symbol MX_Alps_Hybrid:MX-NoLED
- added MX13: MX-NoLED Z, Button_Switch_Keyboard:SW_Cherry_MX_1.00u_PCB, symbol MX_Alps_Hybrid:MX-NoLED
- added MX14: MX-NoLED 2, Button_Switch_Keyboard:SW_Cherry_MX_1.00u_PCB, symbol MX_Alps_Hybrid:MX-NoLED
- added MX15: MX-NoLED W, Button_Switch_Keyboard:SW_Cherry_MX_1.00u_PCB, symbol MX_Alps_Hybrid:MX-NoLED
- added MX16: MX-NoLED S, Button_Switch_Keyboard:SW_Cherry_MX_1.00u_PCB, symbol MX_Alps_Hybrid:MX-NoLED
- added MX17: MX-NoLED F2, Button_Switch_Keyboard:SW_Cherry_MX_1.00u_PCB, symbol MX_Alps_Hybrid:MX-NoLED
- added MX18: MX-NoLED X, Button_Switch_Keyboard:SW_Cherry_MX_1.00u_PCB, symbol MX_Alps_Hybrid:MX-NoLED
- added MX19: MX-NoLED 3, Button_Switch_Keyboard:SW_Cherry_MX_1.00u_PCB, symbol MX_Alps_Hybrid:MX-NoLED
- added MX2: MX-NoLED CRTL, Button_Switch_Keyboard:SW_Cherry_MX_1.25u_PCB, symbol MX_Alps_Hybrid:MX-NoLED
- added MX20: MX-NoLED E, Button_Switch_Keyboard:SW_Cherry_MX_1.00u_PCB, symbol MX_Alps_Hybrid:MX-NoLED
- added MX21: MX-NoLED D, Button_Switch_Keyboard:SW_Cherry_MX_1.00u_PCB, symbol MX_Alps_Hybrid:MX-NoLED
- added MX22: MX-NoLED F3, Button_Switch_Keyboard:SW_Cherry_MX_1.00u_PCB, symbol MX_Alps_Hybrid:MX-NoLED
- added MX23: MX-NoLED C, Button_Switch_Keyboard:SW_Cherry_MX_1.00u_PCB, symbol MX_Alps_Hybrid:MX-NoLED
- added MX24: MX-NoLED 4, Button_Switch_Keyboard:SW_Cherry_MX_1.00u_PCB, symbol MX_Alps_Hybrid:MX-NoLED
- added MX25: MX-NoLED R, Button_Switch_Keyboard:SW_Cherry_MX_1.00u_PCB, symbol MX_Alps_Hybrid:MX-NoLED
- added MX26: MX-NoLED F, Button_Switch_Keyboard:SW_Cherry_MX_1.00u_PCB, symbol MX_Alps_Hybrid:MX-NoLED
- added MX27: MX-NoLED F4, Button_Switch_Keyboard:SW_Cherry_MX_1.00u_PCB, symbol MX_Alps_Hybrid:MX-NoLED
- added MX28: MX-NoLED V, Button_Switch_Keyboard:SW_Cherry_MX_1.00u_PCB, symbol MX_Alps_Hybrid:MX-NoLED
- added MX29: MX-NoLED 5, Button_Switch_Keyboard:SW_Cherry_MX_1.00u_PCB, symbol MX_Alps_Hybrid:MX-NoLED
- added MX3: MX-NoLED Tab, Button_Switch_Keyboard:SW_Cherry_MX_1.50u_PCB, symbol MX_Alps_Hybrid:MX-NoLED
- added MX30: MX-NoLED T, Button_Switch_Keyboard:SW_Cherry_MX_1.00u_PCB, symbol MX_Alps_Hybrid:MX-NoLED
- added MX31: MX-NoLED G, Button_Switch_Keyboard:SW_Cherry_MX_1.00u_PCB, symbol MX_Alps_Hybrid:MX-NoLED
- added MX32: MX-NoLED B, Button_Switch_Keyboard:SW_Cherry_MX_1.00u_PCB, symbol MX_Alps_Hybrid:MX-NoLED
- added MX33: MX-NoLED 6, Button_Switch_Keyboard:SW_Cherry_MX_1.00u_PCB, symbol MX_Alps_Hybrid:MX-NoLED
- added MX34: MX-NoLED F5, Button_Switch_Keyboard:SW_Cherry_MX_1.00u_PCB, symbol MX_Alps_Hybrid:MX-NoLED
- added MX35: MX-NoLED Y, Button_Switch_Keyboard:SW_Cherry_MX_1.00u_PCB, symbol MX_Alps_Hybrid:MX-NoLED
- added MX36: MX-NoLED H, Button_Switch_Keyboard:SW_Cherry_MX_1.00u_PCB, symbol MX_Alps_Hybrid:MX-NoLED
- added MX37: MX-NoLED SPACE, Button_Switch_Keyboard:SW_Cherry_MX_6.25u_PCB, symbol MX_Alps_Hybrid:MX-NoLED
- added MX38: MX-NoLED N, Button_Switch_Keyboard:SW_Cherry_MX_1.00u_PCB, symbol MX_Alps_Hybrid:MX-NoLED
- added MX39: MX-NoLED 7, Button_Switch_Keyboard:SW_Cherry_MX_1.00u_PCB, symbol MX_Alps_Hybrid:MX-NoLED
- added MX4: MX-NoLED CAPS, Button_Switch_Keyboard:SW_Cherry_MX_1.75u_PCB, symbol MX_Alps_Hybrid:MX-NoLED
- added MX40: MX-NoLED F6, Button_Switch_Keyboard:SW_Cherry_MX_1.00u_PCB, symbol MX_Alps_Hybrid:MX-NoLED
- added MX41: MX-NoLED U, Button_Switch_Keyboard:SW_Cherry_MX_1.00u_PCB, symbol MX_Alps_Hybrid:MX-NoLED
- added MX42: MX-NoLED J, Button_Switch_Keyboard:SW_Cherry_MX_1.00u_PCB, symbol MX_Alps_Hybrid:MX-NoLED
- added MX43: MX-NoLED M, Button_Switch_Keyboard:SW_Cherry_MX_1.00u_PCB, symbol MX_Alps_Hybrid:MX-NoLED
- added MX44: MX-NoLED 8, Button_Switch_Keyboard:SW_Cherry_MX_1.00u_PCB, symbol MX_Alps_Hybrid:MX-NoLED
- added MX45: MX-NoLED F7, Button_Switch_Keyboard:SW_Cherry_MX_1.00u_PCB, symbol MX_Alps_Hybrid:MX-NoLED
- added MX46: MX-NoLED I, Button_Switch_Keyboard:SW_Cherry_MX_1.00u_PCB, symbol MX_Alps_Hybrid:MX-NoLED
- added MX47: MX-NoLED K, Button_Switch_Keyboard:SW_Cherry_MX_1.00u_PCB, symbol MX_Alps_Hybrid:MX-NoLED
- added MX48: MX-NoLED ,, Button_Switch_Keyboard:SW_Cherry_MX_1.00u_PCB, symbol MX_Alps_Hybrid:MX-NoLED
- added MX49: MX-NoLED 9, Button_Switch_Keyboard:SW_Cherry_MX_1.00u_PCB, symbol MX_Alps_Hybrid:MX-NoLED
- added MX50: MX-NoLED F8, Button_Switch_Keyboard:SW_Cherry_MX_1.00u_PCB, symbol MX_Alps_Hybrid:MX-NoLED
- added MX51: MX-NoLED O, Button_Switch_Keyboard:SW_Cherry_MX_1.00u_PCB, symbol MX_Alps_Hybrid:MX-NoLED
- added MX52: MX-NoLED L, Button_Switch_Keyboard:SW_Cherry_MX_1.00u_PCB, symbol MX_Alps_Hybrid:MX-NoLED
- added MX53: MX-NoLED ., Button_Switch_Keyboard:SW_Cherry_MX_1.00u_PCB, symbol MX_Alps_Hybrid:MX-NoLED
- added MX54: MX-NoLED 0, Button_Switch_Keyboard:SW_Cherry_MX_1.00u_PCB, symbol MX_Alps_Hybrid:MX-NoLED
- added MX55: MX-NoLED P, Button_Switch_Keyboard:SW_Cherry_MX_1.00u_PCB, symbol MX_Alps_Hybrid:MX-NoLED
- added MX56: MX-NoLED ;, Button_Switch_Keyboard:SW_Cherry_MX_1.00u_PCB, symbol MX_Alps_Hybrid:MX-NoLED
- added MX58: MX-NoLED F9, Button_Switch_Keyboard:SW_Cherry_MX_1.00u_PCB, symbol MX_Alps_Hybrid:MX-NoLED
- added MX59: MX-NoLED /, Button_Switch_Keyboard:SW_Cherry_MX_1.00u_PCB, symbol MX_Alps_Hybrid:MX-NoLED
- added MX60: MX-NoLED dash, Button_Switch_Keyboard:SW_Cherry_MX_1.00u_PCB, symbol MX_Alps_Hybrid:MX-NoLED
- added MX61: MX-NoLED [, Button_Switch_Keyboard:SW_Cherry_MX_1.00u_PCB, symbol MX_Alps_Hybrid:MX-NoLED
- added MX62: MX-NoLED ', Button_Switch_Keyboard:SW_Cherry_MX_1.00u_PCB, symbol MX_Alps_Hybrid:MX-NoLED
- added MX63, MX7: MX-NoLED WIN, Button_Switch_Keyboard:SW_Cherry_MX_1.25u_PCB, symbol MX_Alps_Hybrid:MX-NoLED
- added MX64: MX-NoLED F10, Button_Switch_Keyboard:SW_Cherry_MX_1.00u_PCB, symbol MX_Alps_Hybrid:MX-NoLED
- added MX65: MX-NoLED =, Button_Switch_Keyboard:SW_Cherry_MX_1.00u_PCB, symbol MX_Alps_Hybrid:MX-NoLED
- added MX66: MX-NoLED ], Button_Switch_Keyboard:SW_Cherry_MX_1.00u_PCB, symbol MX_Alps_Hybrid:MX-NoLED
- added MX67: MX-NoLED MENU, Button_Switch_Keyboard:SW_Cherry_MX_1.25u_PCB, symbol MX_Alps_Hybrid:MX-NoLED
- added MX68: MX-NoLED F11, Button_Switch_Keyboard:SW_Cherry_MX_1.00u_PCB, symbol MX_Alps_Hybrid:MX-NoLED
- added MX69: MX-NoLED CTRL, Button_Switch_Keyboard:SW_Cherry_MX_1.25u_PCB, symbol MX_Alps_Hybrid:MX-NoLED
- added MX70: MX-NoLED \\, Button_Switch_Keyboard:SW_Cherry_MX_1.50u_PCB, symbol MX_Alps_Hybrid:MX-NoLED
- added MX71: MX-NoLED ENTER, Button_Switch_Keyboard:SW_Cherry_MX_2.25u_PCB, symbol MX_Alps_Hybrid:MX-NoLED
- added MX72: MX-NoLED R SHIFT, Button_Switch_Keyboard:SW_Cherry_MX_2.75u_PCB, symbol MX_Alps_Hybrid:MX-NoLED
- added MX73: MX-NoLED F12, Button_Switch_Keyboard:SW_Cherry_MX_1.00u_PCB, symbol MX_Alps_Hybrid:MX-NoLED
- added MX74: MX-NoLED BACKSPACE, Button_Switch_Keyboard:SW_Cherry_MX_2.00u_PCB, symbol MX_Alps_Hybrid:MX-NoLED
- added MX75: MX-NoLED LEFT, Button_Switch_Keyboard:SW_Cherry_MX_1.00u_PCB, symbol MX_Alps_Hybrid:MX-NoLED
- added MX76: MX-NoLED Insert, Button_Switch_Keyboard:SW_Cherry_MX_1.00u_PCB, symbol MX_Alps_Hybrid:MX-NoLED
- added MX77: MX-NoLED Delete, Button_Switch_Keyboard:SW_Cherry_MX_1.00u_PCB, symbol MX_Alps_Hybrid:MX-NoLED
- added MX78: MX-NoLED DOWN, Button_Switch_Keyboard:SW_Cherry_MX_1.00u_PCB, symbol MX_Alps_Hybrid:MX-NoLED
- added MX79: MX-NoLED UP, Button_Switch_Keyboard:SW_Cherry_MX_1.00u_PCB, symbol MX_Alps_Hybrid:MX-NoLED
- added MX80: MX-NoLED Home, Button_Switch_Keyboard:SW_Cherry_MX_1.00u_PCB, symbol MX_Alps_Hybrid:MX-NoLED
- added MX81: MX-NoLED End, Button_Switch_Keyboard:SW_Cherry_MX_1.00u_PCB, symbol MX_Alps_Hybrid:MX-NoLED
- added MX82: MX-NoLED RIGHT, Button_Switch_Keyboard:SW_Cherry_MX_1.00u_PCB, symbol MX_Alps_Hybrid:MX-NoLED
- added MX83: MX-NoLED PgUp, Button_Switch_Keyboard:SW_Cherry_MX_1.00u_PCB, symbol MX_Alps_Hybrid:MX-NoLED
- added MX84: MX-NoLED PgDn, Button_Switch_Keyboard:SW_Cherry_MX_1.00u_PCB, symbol MX_Alps_Hybrid:MX-NoLED
- added MX9: MX-NoLED Q, Button_Switch_Keyboard:SW_Cherry_MX_1.00u_PCB, symbol MX_Alps_Hybrid:MX-NoLED
- added R3, R4: 0, Resistor_SMD:R_0805_2012Metric, symbol Device:R
- added R5: 4.7k, Resistor_SMD:R_0805_2012Metric, symbol Device:R
- added R6: 10k, Resistor_SMD:R_0805_2012Metric, symbol Device:R
- added S1: TS-1187A-B-A-B, TS:SW_TS-1187A-B-A-B, symbol TS-1187A-B-A-B:TS-1187A-B-A-B
- added SSD1306: Conn_01x04_Male, Connector_PinHeader_2.54mm:PinHeader_1x04_P2.54mm_Vertical, symbol Connector:Conn_01x04_Male
- added SW1: Rotary_Encoder_Switch, Rotary_Encoder:RotaryEncoder_Alps_EC11E-Switch_Vertical_H20mm, symbol Device:Rotary_Encoder_Switch
- added U1: AMS1117, Package_TO_SOT_SMD:SOT-223-3_TabPin2, symbol Regulator_Linear:AMS1117
- C4, C5: renamed from C?; footprint (none) -> Capacitor_SMD:C_0805_2012Metric
- D10, D15, D6, D7: renamed from D?; footprint (none) -> Diode_SMD:D_SOD-123
- F1: renamed from F?; footprint (none) -> Fuse:Fuse_1206_3216Metric
- MX11: renamed from MX?; value MX-NoLED -> MX-NoLED F1; footprint (none) -> Button_Switch_Keyboard:SW_Cherry_MX_1.00u_PCB
- MX5: renamed from MX?; value MX-NoLED -> MX-NoLED tilde; footprint (none) -> Button_Switch_Keyboard:SW_Cherry_MX_1.00u_PCB
- MX6: renamed from MX?; value MX-NoLED -> MX-NoLED ESC; footprint (none) -> Button_Switch_Keyboard:SW_Cherry_MX_1.00u_PCB
- MX8: renamed from MX?; value MX-NoLED -> MX-NoLED 1; footprint (none) -> Button_Switch_Keyboard:SW_Cherry_MX_1.00u_PCB
- R1, R2, R7, R8: renamed from R?; footprint (none) -> Resistor_SMD:R_0805_2012Metric
- U2: renamed from U?; footprint (none) -> random-keyboard-parts:SOT143B
- USB1: renamed from USB?; footprint (none) -> Type-C:HRO-TYPE-C-31-M-12
- Y1: renamed from Y?; footprint (none) -> Crystal:Crystal_SMD_3225-4Pin_3.2x2.5mm
- gave numbers to parts that had none: 1
Connections:
- net labels added: +3V3, Col1, Col10, Col11, Col12, Col13, Col14, Col15, Col16, Col17, Col2, Col3, Col4, Col5, Col6, Col7, Col8, Col9, ENC_A, ENC_B, ENC_SW, Row1, Row2, Row3, Row4, Row5, Row6, SCL, SDA, SWCLK, SWDIO, SWO, VBUS
- net labels removed: VCC
- wire segments 102 -> 485
- no-connect marks 0 -> 18
Other:
- note added: "MCU decoupling capacitors"
- note added: "OLED I2C"
- note added: "Rotary Encoder"
- note added: "ST-Link"
- note added: "USB C Connector"
- note added: "Voltage regulator"
- note removed: "Decoupling Capacitors"
