File: KiCad Files/custom_keyboard.kicad_pcb (KiCad board)
At the start: 2 copper layers, 199 parts, among them J1 Conn_01x05_Male, SW1 Rotary_Encoder_Switch, U1 AMS1117, U2 PRTR5V0U2X, U3 STM32F401RCTx, Y1 16MHz

Commit message: Col and row routing
Parts:
- C1, C10, C11, C12, C13, C2, C3, C4, C5, C6, C7, C8, C9, F1, J1, R1, R2, R3, R4, R5, R6, R7, R8, S1, U2, Y1: moved to B.Cu
- SW1: value Rotary_Encoder_Switch -> RotaryEncoder_Switch
- moved C3 129.5 mm to (229.6, 43.2)
- moved C8 57.2 mm to (154.9, 163.8), turned to 90 degrees
- moved R7 56.2 mm to (177.8, 154.9), turned to 90 degrees
- moved C6 48.3 mm to (151.1, 158.8)
- moved C13 45.7 mm to (143.5, 154.9)
- moved C11 44.6 mm to (147.3, 154.9)
- moved C2 43.4 mm to (100.8, 157.7)
- moved C9 43.3 mm to (151.1, 154.9)
- moved C7 43.2 mm to (151.1, 162.6)
- moved U1 43.0 mm to (107.3, 153.9)
- moved C1 42.9 mm to (100.8, 152.6)
- moved C12 40.7 mm to (143.5, 158.8)
- moved C10 39.5 mm to (147.3, 158.8)
- moved C4 30.2 mm to (144.8, 149.9)
- moved R6 13.7 mm to (165.1, 148.6)
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Connections:
- C1 pad 2: +5V -> GND
- C10 pad 2: +5V -> GND
- C11 pad 2: +5V -> GND
- C12 pad 2: +5V -> GND
- C13 pad 2: +5V -> GND
- C2 pad 2: +5V -> GND
- C3 pad 1: +5V -> GND
- C4 pad 1: +5V -> GND
- C5 pad 1: +5V -> GND
- C6 pad 2: +5V -> GND
- C7 pad 2: +5V -> GND
- C8 pad 2: +5V -> GND
- C9 pad 2: +5V -> GND
- J1 pad 1: +5V -> GND
- R1 pad 2: +5V -> GND
- R2 pad 2: +5V -> GND
- R4 pad 2: +5V -> GND
- S1 pad A: +5V -> GND
- S1 pad B: +5V -> GND
- SSD1306 pad 1: +5V -> GND
- SW1 pad C: +5V -> GND
- SW1 pad S2: +5V -> GND
- U1 pad 1: +5V -> GND
- U2 pad 1: +5V -> GND
- U3 pad 12: +5V -> GND
- U3 pad 13: Net-(U3-Pad13) -> unconnected-(U3-Pad13)
- U3 pad 18: +5V -> GND
- U3 pad 26: Net-(U3-Pad26) -> unconnected-(U3-Pad26)
- U3 pad 27: Net-(U3-Pad27) -> unconnected-(U3-Pad27)
- U3 pad 28: Net-(U3-Pad28) -> unconnected-(U3-Pad28)
- U3 pad 29: Net-(U3-Pad29) -> unconnected-(U3-Pad29)
- U3 pad 31: +5V -> GND
- U3 pad 33: Net-(U3-Pad33) -> unconnected-(U3-Pad33)
- U3 pad 34: Net-(U3-Pad34) -> unconnected-(U3-Pad34)
- U3 pad 35: Net-(U3-Pad35) -> unconnected-(U3-Pad35)
- U3 pad 36: Net-(U3-Pad36) -> unconnected-(U3-Pad36)
- U3 pad 43: Net-(U3-Pad43) -> unconnected-(U3-Pad43)
- U3 pad 47: +5V -> GND
- U3 pad 50: Net-(U3-Pad50) -> unconnected-(U3-Pad50)
- U3 pad 54: Net-(U3-Pad54) -> unconnected-(U3-Pad54)
- U3 pad 56: Net-(U3-Pad56) -> unconnected-(U3-Pad56)
- U3 pad 57: Net-(U3-Pad57) -> unconnected-(U3-Pad57)
- U3 pad 61: Net-(U3-Pad61) -> unconnected-(U3-Pad61)
- U3 pad 62: Net-(U3-Pad62) -> unconnected-(U3-Pad62)
- U3 pad 63: +5V -> GND
- USB1 pad 1: +5V -> GND
- USB1 pad 12: +5V -> GND
- USB1 pad 13: +5V -> GND
- USB1 pad 3: Net-(USB1-Pad3) -> unconnected-(USB1-Pad3)
- USB1 pad 9: Net-(USB1-Pad9) -> unconnected-(USB1-Pad9)
- Y1 pad 2: +5V -> GND
- Y1 pad 4: +5V -> GND
Routing:
- net Row2: track 0.00 -> 346.4 mm
- net Row1: track 0.00 -> 340.3 mm
- net Row5: track 0.00 -> 317.9 mm
- net Row3: track 0.00 -> 276.4 mm
- net Row4: track 0.00 -> 265.1 mm
- net Row6: track 0.00 -> 264.6 mm
- net Col11: track 0.00 -> 119.5 mm
- net Col13: track 0.00 -> 119.1 mm
- net Col14: track 0.00 -> 113.1 mm
- net Col3: track 0.00 -> 110.3 mm
- net Col10: track 0.00 -> 109.4 mm
- net Col1: track 0.00 -> 104.1 mm
- net Col2: track 0.00 -> 97.1 mm
- net Col15: track 0.00 -> 96.6 mm
- net Col17: track 0.00 -> 95.2 mm
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Other:
- net class Default removed

Commit message: Added outline
Parts:
- moved C3 172.4 mm to (93.9, 149.5)
- moved S1 170.8 mm to (94.2, 154.8)
- moved J1 168.7 mm to (77.2, 154.7)
- moved R1 146.8 mm to (37.7, 54.2)
- moved R2 146.7 mm to (37.8, 58.7)
- moved USB1 145.1 mm to (30.4, 50.2)
- moved U2 137.7 mm to (28.7, 64.0)
- moved F1 123.1 mm to (35.7, 63.5)
Other:
- board outline added: 346.9 x 118.3 mm
Changed lines of the file:
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@@
     )
     (pad_to_mask_clearance 0)
+    (grid_origin 2.2225 165.4175)
     (pcbplotparams
       (layerselection 0x00010fc_ffffffff)
@@
   )
   (footprint "Capacitor_SMD:C_0805_2012Metric" (layer "B.Cu")
-    (at 229.55 43.18)
+    (at 93.8784 149.5044)
     (descr "Capacitor SMD 0805 (2012 Metric), square (rectangular) end terminal, IPC_7351 nominal, (Body size source: IPC-SM-782 page 76, https://www.pcb-3d.com/wordpress/wp-content/uploads/ipc-sm-782a_amendment_1_and_2.pdf, https://docs.google.com/spreadsheets/d/1BsfQQcO9C6DZCsRaXUlFlo91Tg2WpOkGARC1WS5S8t0/edit?usp=sharing), generated with kicad-footprint-generator")
     (tags "capacitor")
@@
   )
   (footprint "Fuse:Fuse_1206_3216Metric" (layer "B.Cu")
-    (at 157.48 45.72 -90)
+    (at 35.6616 63.5381 -90)
     (descr "Fuse SMD 1206 (3216 Metric), square (rectangular) end terminal, IPC_7351 nominal, (Body size source: http://www.tortai-tech.com/upload/download/2011102023233369053.pdf), generated with kicad-footprint-generator")
     (tags "fuse")
@@
   )
   (footprint "Connector_PinHeader_2.54mm:PinHeader_1x05_P2.54mm_Vertical" (layer "B.Cu")
-    (at 204.7875 44.45 -90)
+    (at 77.1702 154.7368 -90)
     (descr "Through hole straight pin header, 1x05, 2.54mm pitch, single row")
     (tags "Through hole pin header THT 1x05 2.54mm single row")
@@
   )
   (footprint "Resistor_SMD:R_0805_2012Metric" (layer "B.Cu")
-    (at 184.15 43.18)
+    (at 37.7444 54.1909)
     (descr "Resistor SMD 0805 (2012 Metric), square (rectangular) end terminal, IPC_7351 nominal, (Body size source: IPC-SM-782 page 72, https://www.pcb-3d.com/wordpress/wp-content/uploads/ipc-sm-782a_amendment_1_and_2.pdf), generated with kicad-footprint-generator")
     (tags "resistor")
@@
   )
   (footprint "Resistor_SMD:R_0805_2012Metric" (layer "B.Cu")
-    (at 184.15 48.26)
+    (at 37.846 58.7121)
     (descr "Resistor SMD 0805 (2012 Metric), square (rectangular) end terminal, IPC_7351 nominal, (Body size source: IPC-SM-782 page 72, https://www.pcb-3d.com/wordpress/wp-content/uploads/ipc-sm-782a_amendment_1_and_2.pdf), generated with kicad-footprint-generator")
     (tags "resistor")
@@
   )
   (footprint "TS:SW_TS-1187A-B-A-B" (layer "B.Cu")
-    (at 223.8375 43.65625)
+    (at 94.1651 154.7876)
     (property "MANUFACTURER" "XKB Industrial Precision")
     (property "MAXIMUM_PACKAGE_HEIGHT" "1.5mm")
@@
   )
   (footprint "random-keyboard-parts:SOT143B" (layer "B.Cu")
-    (at 165.1 45.72)
+    (at 28.6512 63.9953)
     (property "Sheetfile" "C:/Users/kalis/OneDrive/Desktop/keyboard/keyboard_tutorial-main/KiCad Files/custom_keyboard.sch")
     (property "Sheetname" "")
@@
   )
   (footprint "Type-C:HRO-TYPE-C-31-M-12" (layer "B.Cu")
-    (at 175.26 41.275)
+    (at 30.4292 50.2075)
     (property "Sheetfile" "C:/Users/kalis/OneDrive/Desktop/keyboard/keyboard_tutorial-main/KiCad Files/custom_keyboard.sch")
     (property "Sheetname" "")
@@
     )
   )
+  (gr_line (start 347.50375 51.1175) (end 36.35375 51.1175) (layer "Edge.Cuts") (width 0.05))
+  (gr_line (start 349.09125 167.79875) (end 349.09125 52.705) (layer "Edge.Cuts") (width 0.05))
+  (gr_arc (start 3.81 169.38625) (mid 2.687468 168.921282) (end 2.2225 167.79875) (layer "Edge.Cuts") (width 0.05))
+  (gr_arc (start 2.2225 52.705) (mid 2.687468 51.582468) (end 3.81 51.1175) (layer "Edge.Cuts") (width 0.05))
+  (gr_line (start 3.81 169.38625) (end 347.50375 169.38625) (layer "Edge.Cuts") (width 0.05))
+  (gr_line (start 2.2225 52.705) (end 2.2225 167.79875) (layer "Edge.Cuts") (width 0.05))
+  (gr_arc (start 349.09125 167.79875) (mid 348.626282 168.921282) (end 347.50375 169.38625) (layer "Edge.Cuts") (width 0.05))
+  (gr_arc (start 347.50375 51.1175) (mid 348.626282 51.582468) (end 349.09125 52.705) (layer "Edge.Cuts") (width 0.05))
+  (gr_line (start 3.81 51.1175) (end 36.35375 51.1175) (layer "Edge.Cuts") (width 0.05))
   (segment (start 142.875 112.7125) (end 142.875 122.2375) (width 0.254) (layer "F.Cu") (net 11))
   (segment (start 128.74625 74.6125) (end 128.74625 80.764403) (width 0.254) (layer "F.Cu") (net 11))
