File: KiCad Files/custom_keyboard.kicad_sch (KiCad schematic)
At the start: 199 parts, among them SW1 RotaryEncoder_Switch

Commit message: finished routing
Parts:
- removed R3, R4: (no value), symbol Device:R
- added JP1: SolderJumper_3_Open, Jumper:SolderJumper-3_P1.3mm_Open_RoundedPad1.0x1.5mm, symbol Jumper:SolderJumper_3_Open
Connections:
- net +3V3: now also JP1.3 (B)
- net GND: now also JP1.1 (A)
- net at U3.60 (BOOT0): now also JP1.2 (C)
Changed lines of the file:
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@@
   (junction (at 160.02 81.28) (diameter 0) (color 0 0 0 0)
   )
-  (junction (at 326.39 118.11) (diameter 0) (color 0 0 0 0)
-  )
   (junction (at 50.8 143.51) (diameter 0) (color 0 0 0 0)
   )
@@
     (stroke (width 0) (type default) (color 0 0 0 0))
   )
-  (wire (pts (xy 326.39 127) (xy 326.39 128.27))
-    (stroke (width 0) (type default) (color 0 0 0 0))
-  )
   (wire (pts (xy 187.96 55.88) (xy 191.77 55.88))
     (stroke (width 0) (type default) (color 0 0 0 0))
@@
     (stroke (width 0) (type default) (color 0 0 0 0))
   )
-  (wire (pts (xy 345.44 115.57) (xy 347.98 115.57))
+  (wire (pts (xy 327.66 115.57) (xy 347.98 115.57))
     (stroke (width 0) (type default) (color 0 0 0 0))
   )
@@
     (stroke (width 0) (type default) (color 0 0 0 0))
   )
-  (wire (pts (xy 326.39 118.11) (xy 326.39 119.38))
-    (stroke (width 0) (type default) (color 0 0 0 0))
-  )
   (wire (pts (xy 119.38 106.68) (xy 119.38 113.03))
     (stroke (width 0) (type default) (color 0 0 0 0))
@@
     (stroke (width 0) (type default) (color 0 0 0 0))
   )
-  (wire (pts (xy 326.39 118.11) (xy 326.39 116.84))
-    (stroke (width 0) (type default) (color 0 0 0 0))
-  )
   (wire (pts (xy 254 210.82) (xy 254 215.9))
     (stroke (width 0) (type default) (color 0 0 0 0))
@@
     (stroke (width 0) (type default) (color 0 0 0 0))
   )
-  (wire (pts (xy 345.44 118.11) (xy 345.44 115.57))
-    (stroke (width 0) (type default) (color 0 0 0 0))
-  )
   (wire (pts (xy 99.06 106.68) (xy 106.68 106.68))
     (stroke (width 0) (type default) (color 0 0 0 0))
@@
     (stroke (width 0) (type default) (color 0 0 0 0))
   )
-  (wire (pts (xy 326.39 118.11) (xy 345.44 118.11))
-    (stroke (width 0) (type default) (color 0 0 0 0))
-  )
   (wire (pts (xy 228.6 50.8) (xy 228.6 113.03))
     (stroke (width 0) (type default) (color 0 0 0 0))
@@
     (pin "D")
   )
-  (symbol (lib_id "Device:R") (at 326.39 113.03 0) (unit 1)
+  (symbol (lib_id "power:+3V3") (at 323.85 110.49 0) (unit 1)
     (in_bom yes) (on_board yes)
-    (property "Reference" "R3" (id 0) (at 328.168 111.8616 0)
-      (effects (font (size 1.27 1.27)) (justify left))
-    )
-    (property "Value" "" (id 1) (at 328.168 114.173 0)
-      (effects (font (size 1.27 1.27)) (justify left))
-    )
-    (property "Footprint" "" (id 2) (at 324.612 113.03 90)
+    (property "Reference" "#PWR018" (id 0) (at 323.85 114.3 0)
       (effects (font (size 1.27 1.27)) hide)
     )
-    (property "Datasheet" "~" (id 3) (at 326.39 113.03 0)
+    (property "Value" "" (id 1) (at 326.39 110.49 0))
+    (property "Footprint" "" (id 2) (at 323.85 110.49 0)
       (effects (font (size 1.27 1.27)) hide)
     )
-    (pin "1")
-    (pin "2")
-  )
-  (symbol (lib_id "Device:R") (at 326.39 123.19 0) (unit 1)
-    (in_bom yes) (on_board yes)
-    (property "Reference" "R4" (id 0) (at 328.168 122.0216 0)
-      (effects (font (size 1.27 1.27)) (justify left))
-    )
-    (property "Value" "" (id 1) (at 328.168 124.333 0)
-      (effects (font (size 1.27 1.27)) (justify left))
-    )
-    (property "Footprint" "" (id 2) (at 324.612 123.19 90)
-      (effects (font (size 1.27 1.27)) hide)
-    )
-    (property "Datasheet" "~" (id 3) (at 326.39 123.19 0)
-      (effects (font (size 1.27 1.27)) hide)
-    )
-    (pin "1")
-    (pin "2")
-  )
-  (symbol (lib_id "power:+3V3") (at 326.39 109.22 0) (unit 1)
-    (in_bom yes) (on_board yes)
-    (property "Reference" "#PWR018" (id 0) (at 326.39 113.03 0)
-      (effects (font (size 1.27 1.27)) hide)
-    )
-    (property "Value" "" (id 1) (at 328.93 109.22 0))
-    (property "Footprint" "" (id 2) (at 326.39 109.22 0)
-      (effects (font (size 1.27 1.27)) hide)
-    )
-    (property "Datasheet" "" (id 3) (at 326.39 109.22 0)
+    (property "Datasheet" "" (id 3) (at 323.85 110.49 0)
       (effects (font (size 1.27 1.27)) hide)
     )
@@
     (pin "9")
   )
-  (symbol (lib_id "power:GND") (at 326.39 128.27 0) (unit 1)
+  (symbol (lib_id "power:GND") (at 323.85 120.65 0) (unit 1)
     (in_bom yes) (on_board yes) (fields_autoplaced)
-    (property "Reference" "#PWR0105" (id 0) (at 326.39 134.62 0)
+    (property "Reference" "#PWR0105" (id 0) (at 323.85 127 0)
       (effects (font (size 1.27 1.27)) hide)
     )
-    (property "Value" "GND" (id 1) (at 326.39 132.7134 0))
-    (property "Footprint" "" (id 2) (at 326.39 128.27 0)
+    (property "Value" "GND" (id 1) (at 323.85 125.0934 0))
+    (property "Footprint" "" (id 2) (at 323.85 120.65 0)
       (effects (font (size 1.27 1.27)) hide)
     )
-    (property "Datasheet" "" (id 3) (at 326.39 128.27 0)
+    (property "Datasheet" "" (id 3) (at 323.85 120.65 0)
       (effects (font (size 1.27 1.27)) hide)
     )
@@
     (pin "1")
   )
+  (symbol (lib_id "Jumper:SolderJumper_3_Open") (at 323.85 115.57 90) (unit 1)
+    (in_bom yes) (on_board yes)
+    (property "Reference" "JP1" (id 0) (at 322.1991 114.7353 90)
+      (effects (font (size 1.27 1.27)) (justify left))
+    )
+    (property "Value" "SolderJumper_3_Open" (id 1) (at 331.47 127 90)
+      (effects (font (size 1.27 1.27)) (justify left))
+    )
+    (property "Footprint" "Jumper:SolderJumper-3_P1.3mm_Open_RoundedPad1.0x1.5mm" (id 2) (at 323.85 115.57 0)
+      (effects (font (size 1.27 1.27)) hide)
+    )
+    (property "Datasheet" "~" (id 3) (at 323.85 115.57 0)
+      (effects (font (size 1.27 1.27)) hide)
+    )
+    (pin "1")
+    (pin "2")
+    (pin "3")
+  )
   (symbol (lib_id "power:GND") (at 306.07 116.84 0) (unit 1)
     (in_bom yes) (on_board yes) (fields_autoplaced)
@@
       (reference "J1") (unit 1) (value "Conn_01x05_Male") (footprint "Connector_PinHeader_2.54mm:PinHeader_1x05_P2.54mm_Vertical")
     )
+    (path "/6226c47b-6914-4ddb-8595-00bbe052fd0f"
+      (reference "JP1") (unit 1) (value "SolderJumper_3_Open") (footprint "Jumper:SolderJumper-3_P1.3mm_Open_RoundedPad1.0x1.5mm")
+    )
     (path "/00000000-0000-0000-0000-000063111d46"
       (reference "MX1") (unit 1) (value "MX-NoLED L SHIFT") (footprint "Button_Switch_Keyboard:SW_Cherry_MX_2.25u_PCB")
@@
       (reference "R2") (unit 1) (value "5.1k") (footprint "Resistor_SMD:R_0805_2012Metric")
     )
-    (path "/00000000-0000-0000-0000-000065ee0e56"
-      (reference "R3") (unit 1) (value "0") (footprint "Resistor_SMD:R_0805_2012Metric")
-    )
-    (path "/00000000-0000-0000-0000-000065f709c6"
-      (reference "R4") (unit 1) (value "0") (footprint "Resistor_SMD:R_0805_2012Metric")
-    )
     (path "/00000000-0000-0000-0000-000065740a07"

Commit message: Added the 3D Models for all components
Parts:
- C10, C11, C12, C13, C7, C9: value (none) -> 100n; footprint (none) -> Capacitor_SMD:C_0805_2012Metric
- C3: value (none) -> 0.1u; footprint (none) -> Capacitor_SMD:C_0805_2012Metric
- C4, C5: value (none) -> 22p; footprint (none) -> Capacitor_SMD:C_0805_2012Metric
- C6, C8: value (none) -> 4.7u; footprint (none) -> Capacitor_SMD:C_0805_2012Metric
- D1, D10, D101, D102, D103, D105, D107, D108, D110, D111, D113, D115, D116, D117, D119, D12, D120, D121, D123, D125, D126, D127, D129, D130, D131, D14, D15, D17, D19, D20, D22, D24, D25, D27, D28, D3, D30, D32, D33, D35, D36, D38, D4, D40, D41, D43, D44, D46, D48, D5, D50, D51, D52, D54, D56, D58, D6, D60, D61, D62, D64, D66, D68, D69, D7, D70, D72, D73, D76, D77, D78, D80, D82, D84, D85, D87, D89, D9, D91, D92, D94, D95, D97, D99: value (none) -> D_Small; footprint (none) -> Diode_SMD:D_SOD-123
- F1: value (none) -> 500m; footprint (none) -> Fuse:Fuse_1206_3216Metric
- J1: value (none) -> Conn_01x05_Male; footprint (none) -> Connector_PinHeader_2.54mm:PinHeader_1x05_P2.54mm_Vertical
- MX1: value (none) -> MX-NoLED L SHIFT; footprint (none) -> kals_keeb:SW_Cherry_MX_2.25u_PCB
- MX10: value (none) -> MX-NoLED A; footprint (none) -> kals_keeb:SW_Cherry_MX_1.00u_PCB
- MX11: value (none) -> MX-NoLED F1; footprint (none) -> kals_keeb:SW_Cherry_MX_1.00u_PCB
- MX12, MX57: value (none) -> MX-NoLED ALT; footprint (none) -> kals_keeb:SW_Cherry_MX_1.25u_PCB
- MX13: value (none) -> MX-NoLED Z; footprint (none) -> kals_keeb:SW_Cherry_MX_1.00u_PCB
- MX14: value (none) -> MX-NoLED 2; footprint (none) -> kals_keeb:SW_Cherry_MX_1.00u_PCB
- MX15: value (none) -> MX-NoLED W; footprint (none) -> kals_keeb:SW_Cherry_MX_1.00u_PCB
- MX16: value (none) -> MX-NoLED S; footprint (none) -> kals_keeb:SW_Cherry_MX_1.00u_PCB
- MX17: value (none) -> MX-NoLED F2; footprint (none) -> kals_keeb:SW_Cherry_MX_1.00u_PCB
- MX18: value (none) -> MX-NoLED X; footprint (none) -> kals_keeb:SW_Cherry_MX_1.00u_PCB
- MX19: value (none) -> MX-NoLED 3; footprint (none) -> kals_keeb:SW_Cherry_MX_1.00u_PCB
- MX2: value (none) -> MX-NoLED CRTL; footprint (none) -> kals_keeb:SW_Cherry_MX_1.25u_PCB
- MX20: value (none) -> MX-NoLED E; footprint (none) -> kals_keeb:SW_Cherry_MX_1.00u_PCB
- MX21: value (none) -> MX-NoLED D; footprint (none) -> kals_keeb:SW_Cherry_MX_1.00u_PCB
- MX22: value (none) -> MX-NoLED F3; footprint (none) -> kals_keeb:SW_Cherry_MX_1.00u_PCB
- MX23: value (none) -> MX-NoLED C; footprint (none) -> kals_keeb:SW_Cherry_MX_1.00u_PCB
- MX24: value (none) -> MX-NoLED 4; footprint (none) -> kals_keeb:SW_Cherry_MX_1.00u_PCB
- MX25: value (none) -> MX-NoLED R; footprint (none) -> kals_keeb:SW_Cherry_MX_1.00u_PCB
- MX26: value (none) -> MX-NoLED F; footprint (none) -> kals_keeb:SW_Cherry_MX_1.00u_PCB
- MX27: value (none) -> MX-NoLED F4; footprint (none) -> kals_keeb:SW_Cherry_MX_1.00u_PCB
- MX28: value (none) -> MX-NoLED V; footprint (none) -> kals_keeb:SW_Cherry_MX_1.00u_PCB
- MX29: value (none) -> MX-NoLED 5; footprint (none) -> kals_keeb:SW_Cherry_MX_1.00u_PCB
- MX3: value (none) -> MX-NoLED Tab; footprint (none) -> kals_keeb:SW_Cherry_MX_1.50u_PCB
- MX30: value (none) -> MX-NoLED T; footprint (none) -> kals_keeb:SW_Cherry_MX_1.00u_PCB
- MX31: value (none) -> MX-NoLED G; footprint (none) -> kals_keeb:SW_Cherry_MX_1.00u_PCB
- MX32: value (none) -> MX-NoLED B; footprint (none) -> kals_keeb:SW_Cherry_MX_1.00u_PCB
- MX33: value (none) -> MX-NoLED 6; footprint (none) -> kals_keeb:SW_Cherry_MX_1.00u_PCB
- MX34: value (none) -> MX-NoLED F5; footprint (none) -> kals_keeb:SW_Cherry_MX_1.00u_PCB
- MX35: value (none) -> MX-NoLED Y; footprint (none) -> kals_keeb:SW_Cherry_MX_1.00u_PCB
- MX36: value (none) -> MX-NoLED H; footprint (none) -> kals_keeb:SW_Cherry_MX_1.00u_PCB
- MX37: value (none) -> MX-NoLED SPACE; footprint (none) -> kals_keeb:SW_Cherry_MX_6.25u_PCB
- MX38: value (none) -> MX-NoLED N; footprint (none) -> kals_keeb:SW_Cherry_MX_1.00u_PCB
- MX39: value (none) -> MX-NoLED 7; footprint (none) -> kals_keeb:SW_Cherry_MX_1.00u_PCB
- MX4: value (none) -> MX-NoLED CAPS; footprint (none) -> kals_keeb:SW_Cherry_MX_1.75u_PCB
- MX40: value (none) -> MX-NoLED F6; footprint (none) -> kals_keeb:SW_Cherry_MX_1.00u_PCB
- MX41: value (none) -> MX-NoLED U; footprint (none) -> kals_keeb:SW_Cherry_MX_1.00u_PCB
- MX42: value (none) -> MX-NoLED J; footprint (none) -> kals_keeb:SW_Cherry_MX_1.00u_PCB
- MX43: value (none) -> MX-NoLED M; footprint (none) -> kals_keeb:SW_Cherry_MX_1.00u_PCB
- MX44: value (none) -> MX-NoLED 8; footprint (none) -> kals_keeb:SW_Cherry_MX_1.00u_PCB
- MX45: value (none) -> MX-NoLED F7; footprint (none) -> kals_keeb:SW_Cherry_MX_1.00u_PCB
- MX46: value (none) -> MX-NoLED I; footprint (none) -> kals_keeb:SW_Cherry_MX_1.00u_PCB
- MX47: value (none) -> MX-NoLED K; footprint (none) -> kals_keeb:SW_Cherry_MX_1.00u_PCB
- MX48: value (none) -> MX-NoLED ,; footprint (none) -> kals_keeb:SW_Cherry_MX_1.00u_PCB
- MX49: value (none) -> MX-NoLED 9; footprint (none) -> kals_keeb:SW_Cherry_MX_1.00u_PCB
- MX5: value (none) -> MX-NoLED tilde; footprint (none) -> kals_keeb:SW_Cherry_MX_1.00u_PCB
- MX50: value (none) -> MX-NoLED F8; footprint (none) -> kals_keeb:SW_Cherry_MX_1.00u_PCB
- MX51: value (none) -> MX-NoLED O; footprint (none) -> kals_keeb:SW_Cherry_MX_1.00u_PCB
- MX52: value (none) -> MX-NoLED L; footprint (none) -> kals_keeb:SW_Cherry_MX_1.00u_PCB
- MX53: value (none) -> MX-NoLED .; footprint (none) -> kals_keeb:SW_Cherry_MX_1.00u_PCB
- MX54: value (none) -> MX-NoLED 0; footprint (none) -> kals_keeb:SW_Cherry_MX_1.00u_PCB
- MX55: value (none) -> MX-NoLED P; footprint (none) -> kals_keeb:SW_Cherry_MX_1.00u_PCB
- MX56: value (none) -> MX-NoLED ;; footprint (none) -> kals_keeb:SW_Cherry_MX_1.00u_PCB
- MX58: value (none) -> MX-NoLED F9; footprint (none) -> kals_keeb:SW_Cherry_MX_1.00u_PCB
- MX59: value (none) -> MX-NoLED /; footprint (none) -> kals_keeb:SW_Cherry_MX_1.00u_PCB
- MX6: value (none) -> MX-NoLED ESC; footprint (none) -> kals_keeb:SW_Cherry_MX_1.00u_PCB
- MX60: value (none) -> MX-NoLED dash; footprint (none) -> kals_keeb:SW_Cherry_MX_1.00u_PCB
- MX61: value (none) -> MX-NoLED [; footprint (none) -> kals_keeb:SW_Cherry_MX_1.00u_PCB
- MX62: value (none) -> MX-NoLED '; footprint (none) -> kals_keeb:SW_Cherry_MX_1.00u_PCB
- MX63, MX7: value (none) -> MX-NoLED WIN; footprint (none) -> kals_keeb:SW_Cherry_MX_1.25u_PCB
- MX64: value (none) -> MX-NoLED F10; footprint (none) -> kals_keeb:SW_Cherry_MX_1.00u_PCB
- MX65: value (none) -> MX-NoLED =; footprint (none) -> kals_keeb:SW_Cherry_MX_1.00u_PCB
- MX66: value (none) -> MX-NoLED ]; footprint (none) -> kals_keeb:SW_Cherry_MX_1.00u_PCB
- MX67: value (none) -> MX-NoLED MENU; footprint (none) -> kals_keeb:SW_Cherry_MX_1.25u_PCB
- MX68: value (none) -> MX-NoLED F11; footprint (none) -> kals_keeb:SW_Cherry_MX_1.00u_PCB
- MX69: value (none) -> MX-NoLED CTRL; footprint (none) -> kals_keeb:SW_Cherry_MX_1.25u_PCB
- MX70: value (none) -> MX-NoLED \; footprint (none) -> kals_keeb:SW_Cherry_MX_1.50u_PCB
- MX71: value (none) -> MX-NoLED ENTER; footprint (none) -> kals_keeb:SW_Cherry_MX_2.25u_PCB
- MX72: value (none) -> MX-NoLED R SHIFT; footprint (none) -> kals_keeb:SW_Cherry_MX_2.75u_PCB
- MX73: value (none) -> MX-NoLED F12; footprint (none) -> kals_keeb:SW_Cherry_MX_1.00u_PCB
- MX74: value (none) -> MX-NoLED BACKSPACE; footprint (none) -> kals_keeb:SW_Cherry_MX_2.00u_PCB
- MX75: value (none) -> MX-NoLED LEFT; footprint (none) -> kals_keeb:SW_Cherry_MX_1.00u_PCB
- MX76: value (none) -> MX-NoLED Insert; footprint (none) -> kals_keeb:SW_Cherry_MX_1.00u_PCB
- MX77: value (none) -> MX-NoLED Delete; footprint (none) -> kals_keeb:SW_Cherry_MX_1.00u_PCB
- MX78: value (none) -> MX-NoLED DOWN; footprint (none) -> kals_keeb:SW_Cherry_MX_1.00u_PCB
- MX79: value (none) -> MX-NoLED UP; footprint (none) -> kals_keeb:SW_Cherry_MX_1.00u_PCB
- MX8: value (none) -> MX-NoLED 1; footprint (none) -> kals_keeb:SW_Cherry_MX_1.00u_PCB
- MX80: value (none) -> MX-NoLED Home; footprint (none) -> kals_keeb:SW_Cherry_MX_1.00u_PCB
- MX81: value (none) -> MX-NoLED End; footprint (none) -> kals_keeb:SW_Cherry_MX_1.00u_PCB
- MX82: value (none) -> MX-NoLED RIGHT; footprint (none) -> kals_keeb:SW_Cherry_MX_1.00u_PCB
- MX83: value (none) -> MX-NoLED PgUp; footprint (none) -> kals_keeb:SW_Cherry_MX_1.00u_PCB
- MX84: value (none) -> MX-NoLED PgDn; footprint (none) -> kals_keeb:SW_Cherry_MX_1.00u_PCB
- MX9: value (none) -> MX-NoLED Q; footprint (none) -> kals_keeb:SW_Cherry_MX_1.00u_PCB
- R1, R2: value (none) -> 5.1k; footprint (none) -> Resistor_SMD:R_0805_2012Metric
- R5: value (none) -> 4.7k; footprint (none) -> Resistor_SMD:R_0805_2012Metric
- R6: value (none) -> 10k; footprint (none) -> Resistor_SMD:R_0805_2012Metric
- R7, R8: value (none) -> 22; footprint (none) -> Resistor_SMD:R_0805_2012Metric
- S1: value (none) -> TS-1187A-B-A-B; footprint (none) -> TS:SW_TS-1187A-B-A-B
- SSD1306: value (none) -> Conn_01x04_Male; footprint (none) -> Connector_PinHeader_2.54mm:PinHeader_1x04_P2.54mm_Vertical
- SW1: footprint Rotary_Encoder:RotaryEncoder_Alps_EC11E-Switch_Vertical_H20mm -> kals_keeb:RotaryEncoder_Alps_EC11E_Vertical_H20mm
- U1: value (none) -> AMS1117; footprint (none) -> Package_TO_SOT_SMD:SOT-223-3_TabPin2
- U2: value (none) -> PRTR5V0U2X; footprint (none) -> random-keyboard-parts:SOT143B
- U3: value (none) -> STM32F401RCTx; footprint (none) -> Package_QFP:LQFP-64_10x10mm_P0.5mm
- USB1: footprint Type-C:HRO-TYPE-C-31-M-12 -> kals_keeb:USB_C_Receptacle_HRO_TYPE-C-31-M-12
- Y1: value (none) -> 16MHz; footprint (none) -> Crystal:Crystal_SMD_3225-4Pin_3.2x2.5mm
